Commit message: removes self-collision for now

File: controllers/resources/iiwa14_spheres_dense_elbow_collision.urdf (robot description, URDF)
Before this commit: robot iiwa14, 10 links, 9 joints
Links:
- link iiwa_link_0: geometry visual mesh filename=package://drake_models/iiwa_description/meshes/iiwa14/visua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
- link iiwa_link_1: geometry visual mesh filename=package://drake_models/iiwa_description/meshes/iiwa14/visua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
- link iiwa_link_2: geometry visual mesh filename=package://drake_models/iiwa_description/meshes/iiwa14/visua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; visual mesh filename=package://drake_models/iiwa_description/meshes/iiwa14/visua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
- link iiwa_link_3: geometry visual mesh filename=package://drake_models/iiwa_description/meshes/iiwa14/visua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; visual mesh filename=package://drake_models/iiwa_description/meshes/iiwa14/visua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
- link iiwa_link_4: geometry visual mesh filename=package://drake_models/iiwa_description/meshes/iiwa14/visua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; visual mesh filename=package://drake_models/iiwa_description/meshes/iiwa14/visua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
- link iiwa_link_6: geometry visual mesh filename=package://drake_models/iiwa_description/meshes/iiwa14/visua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; visual mesh filename=package://drake_models/iiwa_description/meshes/iiwa14/visua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
- link iiwa_link_7: geometry visual mesh filename=package://drake_models/iiwa_description/meshes/iiwa14/visua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
